File: Hardware/APL1/APL1.kicad_pcb (KiCad board)
At the start: 2 copper layers, 0 parts

Commit message: Layout PCB
Parts:
- added C1: 100nF, Capacitor_THT:C_Disc_D5.0mm_W2.5mm_P5.00mm, F.Cu at (72.2, 101.4)
- added C10: 1uF, Capacitor_THT:C_Disc_D5.0mm_W2.5mm_P5.00mm, F.Cu at (98.2, 65.8)
- added C11: 18pF, Capacitor_THT:C_Disc_D5.0mm_W2.5mm_P5.00mm, F.Cu at (189.8, 102.6)
- added C12: 18pF, Capacitor_THT:C_Disc_D5.0mm_W2.5mm_P5.00mm, F.Cu at (189.8, 107.5)
- added C13: 1uF, Capacitor_THT:C_Disc_D5.0mm_W2.5mm_P5.00mm, F.Cu at (114.7, 65.8)
- added C14: 1uF, Capacitor_THT:C_Disc_D5.0mm_W2.5mm_P5.00mm, F.Cu at (98.2, 52.1)
- added C15: 1uF, Capacitor_THT:C_Disc_D5.0mm_W2.5mm_P5.00mm, F.Cu at (102.1, 65.8)
- added C2: 100nF, Capacitor_THT:C_Disc_D5.0mm_W2.5mm_P5.00mm, F.Cu at (150.3, 70.7)
- added C3: 100nF, Capacitor_THT:C_Disc_D5.0mm_W2.5mm_P5.00mm, F.Cu at (150.3, 111.4)
- added C4: 100nF, Capacitor_THT:C_Disc_D5.0mm_W2.5mm_P5.00mm, F.Cu at (176.1, 96.3)
- added C5: 100nF, Capacitor_THT:C_Disc_D5.0mm_W2.5mm_P5.00mm, F.Cu at (192.8, 115.5)
- added C6: 100nF, Capacitor_THT:C_Disc_D5.0mm_W2.5mm_P5.00mm, F.Cu at (98.9, 133.4)
- added C7: 100nF, Capacitor_THT:C_Disc_D5.0mm_W2.5mm_P5.00mm, F.Cu at (150.3, 125.2)
- added C8: 100nF, Capacitor_THT:C_Disc_D5.0mm_W2.5mm_P5.00mm, F.Cu at (150.3, 138.3)
- added C9: 100nF, Capacitor_THT:C_Disc_D5.0mm_W2.5mm_P5.00mm, F.Cu at (65.3, 145.7)
- added D1: POWER LED, LED_THT:LED_D3.0mm, F.Cu at (59.6, 71.0)
- added G***: LOGO, A.C. Wright Logo:A.C. Wright Logo 10mm, F.Cu at (187.2, 89.4)
- added J1: 6502 BUS, 6502 Parts:6502 Bus Connector, F.Cu at (61.0, 132.1)
- added J2: KEYBOARD, Package_DIP:DIP-16_W7.62mm_Socket_LongPads, F.Cu at (155.4, 145.8)
- added J3: DB9 MALE (DTE), Connector_Dsub:DSUB-9_Pins_Horizontal_P2.77x2.84mm_EdgePinOffset7.70mm_Housed_MountingHolesOffset9.12mm, F.Cu at (138.0, 61.4)
- added J4: 5V DC, Connector_BarrelJack:BarrelJack_Horizontal, F.Cu at (68.6, 64.0)
- added J5: PS/2, 6502 Parts:KMDGX-6S-BS, F.Cu at (161.7, 59.8)
- added J6: VIDEO, 6502 Parts:SWITCHCRAFT_PJRAN1X1U0XX, F.Cu at (182.0, 54.8)
- added J7: SERIAL, Connector_PinHeader_2.54mm:PinHeader_1x04_P2.54mm_Horizontal, F.Cu at (104.3, 60.5)
- added R1: 1k, Resistor_THT:R_Axial_DIN0207_L6.3mm_D2.5mm_P10.16mm_Horizontal, F.Cu at (72.2, 127.0)
- added R2: 1k, Resistor_THT:R_Axial_DIN0207_L6.3mm_D2.5mm_P10.16mm_Horizontal, F.Cu at (72.2, 104.1)
- added R3: 1k, Resistor_THT:R_Axial_DIN0207_L6.3mm_D2.5mm_P10.16mm_Horizontal, F.Cu at (68.8, 135.5)
- added R4: 1k, Resistor_THT:R_Axial_DIN0207_L6.3mm_D2.5mm_P10.16mm_Horizontal, F.Cu at (72.2, 135.6)
- added R5: 330, Resistor_THT:R_Axial_DIN0207_L6.3mm_D2.5mm_P10.16mm_Horizontal, F.Cu at (59.6, 68.2)
- added R6: 1k, Resistor_THT:R_Axial_DIN0207_L6.3mm_D2.5mm_P10.16mm_Horizontal, F.Cu at (178.6, 78.5)
- added R7: 820, Resistor_THT:R_Axial_DIN0207_L6.3mm_D2.5mm_P10.16mm_Horizontal, F.Cu at (182.0, 78.5)
- added R8: 820, Resistor_THT:R_Axial_DIN0207_L6.3mm_D2.5mm_P10.16mm_Horizontal, F.Cu at (185.3, 78.5)
- added REF**: MountingHole_3.2mm_M3, MountingHole:MountingHole_3.2mm_M3, F.Cu at (55.0, 145.0)
- added REF**: Polarity_Center_Positive_6mm_SilkScreen, Symbol:Polarity_Center_Positive_6mm_SilkScreen, F.Cu at (75.0, 62.0)
- added REF**: OSHW-Logo2_7.3x6mm_SilkScreen, Symbol:OSHW-Logo2_7.3x6mm_SilkScreen, F.Cu at (68.7, 72.5)
- added REF**: MountingHole_3.2mm_M3, MountingHole:MountingHole_3.2mm_M3, F.Cu at (195.0, 145.0)
- added REF**: MountingHole_3.2mm_M3, MountingHole:MountingHole_3.2mm_M3, F.Cu at (195.0, 55.0)
- added REF**: MountingHole_3.2mm_M3, MountingHole:MountingHole_3.2mm_M3, F.Cu at (55.0, 55.0)
- added SW1: POWER, 6502 Parts:SW_400MSP1R6BLKM6QE, F.Cu at (86.4, 64.0)
- added U1: 74HCT04, Package_DIP:DIP-14_W7.62mm_Socket_LongPads, F.Cu at (104.2, 145.8)
- added U10: ATmega1284-P, Package_DIP:DIP-40_W15.24mm_Socket_LongPads, F.Cu at (155.8, 70.8)
- added U2: 6502, Package_DIP:DIP-40_W15.24mm_Socket_LongPads, F.Cu at (78.5, 85.1)
- added U3: 65C21, Package_DIP:DIP-40_W15.24mm_Socket_LongPads, F.Cu at (104.2, 85.0)
- added U4: AS6C62256, Package_DIP:DIP-28_W15.24mm_Socket_LongPads, F.Cu at (129.8, 70.7)
- added U5: 74HCT00, Package_DIP:DIP-14_W7.62mm_Socket_LongPads, F.Cu at (156.4, 132.8)
- added U6: 74LS138, Package_DIP:DIP-16_W7.62mm_Socket_LongPads, F.Cu at (77.4, 145.9)
- added U7: 28C64, Package_DIP:DIP-28_W15.24mm_Socket_LongPads, F.Cu at (129.8, 111.4)
- added U8: 74HCT245, Package_DIP:DIP-20_W7.62mm_Socket_LongPads, F.Cu at (179.9, 115.5)
- added U9: MAX232, Package_DIP:DIP-16_W7.62mm_Socket_LongPads, F.Cu at (103.2, 78.4)
- added Y1: 1MHz, Oscillator:Oscillator_DIP-14, F.Cu at (78.5, 78.4)
- added Y2: 28.63636MHz, Crystal:Crystal_HC49-U_Vertical, F.Cu at (178.6, 107.5)
Routing:
- added copper zone on B.Cu, net GND
- added copper zone on F.Cu, net GND
Other:
- board outline added: 150 x 100 mm
- board text added: "$A000"
- board text added: "$B000"
- board text added: "$C000"
- board text added: "A0"
- board text added: "A1"
- board text added: "A10"
- board text added: "A11"
- board text added: "A12"
- board text added: "A13"
- board text added: "A14"
- board text added: "A15"
- board text added: "A2"
- board text added: "A3"
- board text added: "A4"
- board text added: "A5"
- board text added: "A6"
- board text added: "A7"
- board text added: "A8"
- board text added: "A9"
- board text added: "APL1"
- board text added: "D0"
- board text added: "D1"
- board text added: "D2"
- board text added: "D3"
- board text added: "D4"
- board text added: "D5"
- board text added: "D6"
- board text added: "D7"
- board text added: "EXP0"
- board text added: "EXP1"
- board text added: "GND"
- board text added: "IRQB"
- board text added: "JLCJLCJLCJLC"
- board text added: "NMIB"
- board text added: "PHI2"
- board text added: "RDY"
- board text added: "RESB"
- board text added: "RWB"
- board text added: "SYNC"
- board text added: "VCC"
- board text added: "© 2026 A.C. Wright Design | acwrightdesign.com | Rev 1.0"
