File: Hardware/APL1/APL1.kicad_sch (KiCad schematic)
At the start: 33 parts, among them J1 6502 Bus, J2 ASCII KEYBOARD, J3 PS/2, J4 VIDEO, J5 SERIAL, U1 6502, U2 65C21, U3 AS6C62256, U4 74LS00, U5 74LS138, U6 28C64, U7 74LS245, U8 ATmega1284-P, Y1 1MHz, Y2 20MHz

Commit message: Update to schematic
Parts:
- removed R7: 75, symbol Device:R
- added C9: 100nF, symbol Device:C_Small
- added U1: 74HC04, symbol 74xx:74HC04
- J2: value ASCII KEYBOARD -> APPLE1 KEYBOARD; symbol Parts:ASCII KEYBOARD -> Parts:APPLE1 KEYBOARD
- R5: value 470 -> 1k
- R6: value 270 -> 470
- renumbered C9 to C10, C10 to C11, C11 to C12, U1 to U2, U2 to U3, U3 to U4, U4 to U5, U5 to U6, U6 to U7, U7 to U8, U8 to U9
Connections:
- net GND: now also J2.9 (GND), C9.2, U1.11, U1.13, U1.3, U1.5, U1.7 (GND), U1.9; no longer J2.8 (GND)
- net KBD0: now also J2.5 (B1); no longer J2.12 (KBD0)
- net KBD1: now also J2.4 (B2); no longer J2.13 (KBD1)
- net KBD2: now also J2.3 (B3); no longer J2.10 (KBD2)
- net KBD3: now also J2.2 (B4); no longer J2.11 (KBD3)
- net KBD5: now also J2.7 (B6); no longer J2.5 (KBD5)
- net KBD6: now also J2.8 (B7); no longer J2.7 (KBD6)
- net KBDSTROBE: now also J2.14 (STROBE); no longer J2.2 (STROBE)
- net RESB: no longer J2.3 (RESET)
- net VCC: now also J2.16 (VCC), C9.1, U1.14 (VCC); no longer J2.1 (VCC)
- net KBDRESB: now reaches U9.18 (PD4)
- net KBDRESB: now also J2.1 (RESET)
- net RDAB: now reaches U9.29 (PC7)
- net RDAB: now also U3.18 (CB1)
- net at U3.19 (CB2): now also U1.1
- net CLRB renamed KBDCLRB
- net KBDCLRB: now also J2.12 (CLEAR); no longer J2.4 (CLEAR)
- net DSPRDY renamed DA
- net DA: now also U1.2
- no-connect marks 19 -> 23
Other:
- moved on the sheet: C11, C12, J3, J4, R1, R2, R3, R4, R5, R6, U8, U9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

Commit message: Layout PCB
Parts:
- removed C9: 100nF, symbol Device:C_Small
- added C10, C13, C14, C15: 1uF, Capacitor_THT:C_Disc_D5.0mm_W2.5mm_P5.00mm, symbol Device:C
- added D1: POWER LED, LED_THT:LED_D3.0mm, symbol Device:LED
- added J3: DB9 MALE (DTE), Connector_Dsub:DSUB-9_Pins_Horizontal_P2.77x2.84mm_EdgePinOffset7.70mm_Housed_MountingHolesOffset9.12mm, symbol Connector:DE9_Pins_MountingHoles
- added J4: 5V DC, Connector_BarrelJack:BarrelJack_Horizontal, symbol Connector:Barrel_Jack_Switch
- added R5: 330, Resistor_THT:R_Axial_DIN0207_L6.3mm_D2.5mm_P10.16mm_Horizontal, symbol Device:R
- added R8: 820, Resistor_THT:R_Axial_DIN0207_L6.3mm_D2.5mm_P10.16mm_Horizontal, symbol Device:R
- added SW1: POWER, 6502 Parts:SW_400MSP1R6BLKM6QE, symbol Switch:SW_SPDT
- added U9: MAX232, Package_DIP:DIP-16_W7.62mm_Socket_LongPads, symbol Interface_UART:MAX232
- C1, C2, C3, C4, C5, C6, C7, C8: footprint (none) -> Capacitor_THT:C_Disc_D5.0mm_W2.5mm_P5.00mm
- C11, C12: value 20pF -> 18pF; footprint (none) -> Capacitor_THT:C_Disc_D5.0mm_W2.5mm_P5.00mm
- C9: renamed from C10; footprint (none) -> Capacitor_THT:C_Disc_D5.0mm_W2.5mm_P5.00mm
- J1: value 6502 Bus -> 6502 BUS; footprint (none) -> 6502 Parts:6502 Bus Connector
- J2: value APPLE1 KEYBOARD -> KEYBOARD; footprint (none) -> Package_DIP:DIP-16_W7.62mm_Socket_LongPads; symbol Parts:APPLE1 KEYBOARD -> 6502 Parts:APPLE1 KEYBOARD
- J5: renamed from J3; footprint (none) -> 6502 Parts:KMDGX-6S-BS; symbol Parts:KMDGX-6S-BS -> 6502 Parts:KMDGX-6S-BS
- J6: renamed from J4; footprint (none) -> 6502 Parts:SWITCHCRAFT_PJRAN1X1U0XX
- J7: renamed from J5; footprint (none) -> Connector_PinHeader_2.54mm:PinHeader_1x04_P2.54mm_Horizontal
- R1, R2, R3, R4: footprint (none) -> Resistor_THT:R_Axial_DIN0207_L6.3mm_D2.5mm_P10.16mm_Horizontal
- R6: renamed from R5; footprint (none) -> Resistor_THT:R_Axial_DIN0207_L6.3mm_D2.5mm_P10.16mm_Horizontal
- R7: renamed from R6; value 470 -> 820; footprint (none) -> Resistor_THT:R_Axial_DIN0207_L6.3mm_D2.5mm_P10.16mm_Horizontal
- U1: value 74HC04 -> 74HCT04; footprint (none) -> Package_DIP:DIP-14_W7.62mm_Socket_LongPads
- U10: renamed from U9; footprint Package_DIP:DIP-40_W15.24mm -> Package_DIP:DIP-40_W15.24mm_Socket_LongPads
- U2: footprint (none) -> Package_DIP:DIP-40_W15.24mm_Socket_LongPads; symbol Parts:6502 -> 6502 Parts:6502
- U3: footprint (none) -> Package_DIP:DIP-40_W15.24mm_Socket_LongPads; symbol Parts:65C21 -> 6502 Parts:65C21
- U4: footprint (none) -> Package_DIP:DIP-28_W15.24mm_Socket_LongPads; symbol Parts:AS6C62256 -> 6502 Parts:AS6C62256
- U5: value 74LS00 -> 74HCT00; footprint (none) -> Package_DIP:DIP-14_W7.62mm_Socket_LongPads
- U6: footprint (none) -> Package_DIP:DIP-16_W7.62mm_Socket_LongPads
- U7: footprint Package_DIP:DIP-28_W15.24mm -> Package_DIP:DIP-28_W15.24mm_Socket_LongPads
- U8: value 74LS245 -> 74HCT245; footprint (none) -> Package_DIP:DIP-20_W7.62mm_Socket_LongPads
- Y2: value 20MHz -> 28.63636MHz; Digikey (none) -> 887-1256-ND
Connections:
- net GND: now also C14.1, C15.1, J3.5, J3.SH (PAD), J4.2, J4.3, R5.2, U9.10 (T2IN), U9.15 (GND), U9.8 (R2IN)
- net RX: now also U9.12 (R1OUT)
- net TX: now also U9.11 (T1IN)
- net VCC: now also D1.2 (A), SW1.1 (A), U9.16 (VCC)
- net at J6.1 (In), R6.2, R7.2: now also R8.2
- net at U10.24 (PC2): now also R8.1
- new net: J4.1, SW1.2 (B)
- new net: D1.1 (K), R5.1
- new net: C13.1, U9.5 (C2-)
- new net: C13.2, U9.4 (C2+)
- new net: C10.1, U9.1 (C1+)
- new net: C14.2, U9.2 (VS+)
- new net: C10.2, U9.3 (C1-)
- new net: C15.2, U9.6 (VS-)
- new net RXIN: J3.2, U9.13 (R1IN)
- new net TXOUT: J3.3, U9.14 (T1OUT)
- no-connect marks 23 -> 31
Other:
- moved on the sheet: C11, C12, J5, J6, J7, R6, R7, U10, U1B, U1C, U1D, U1E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
