File: Hardware/APL1/Rev 1.1/APL1.kicad_pcb (KiCad board)
At the start: 2 copper layers, 150 x 100 mm, 51 parts, among them J1 6502 BUS, J2 KEYBOARD, J3 SERIAL (DTE), J4 5V DC, J5 PS/2, J6 VIDEO, SW1 POWER, U1 74LS04, U10 ATmega1284-P, U2 6502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

Commit message: Add Rev 1.1
Parts:
- added C17: 10uF, Capacitor_THT:CP_Radial_D4.0mm_P1.50mm, F.Cu at (69.1, 78.5)
- added R9: 10k, Resistor_THT:R_Axial_DIN0207_L6.3mm_D2.5mm_P10.16mm_Horizontal, F.Cu at (189.8, 96.3)
- R1, R2, R3, R4: value 1k -> 4.7k
- moved REF** 1.40 mm to (69.8, 71.0)
- turned C4 to 90 degrees
Connections:
- net KBDCLRB renamed KBDCLR
Routing:
- net KBDCLR: track 36.2 -> 78.1 mm, vias 3 -> 5
- net VCC: track 559.2 -> 567.3 mm
- net GND: vias 46 -> 47
Other:
- board text added: "© 2026 A.C. Wright Design | acwrightdesign.com | Rev 1.1"
- board text removed: "© 2026 A.C. Wright Design | acwrightdesign.com | Rev 1.0"
