File: Hardware/APL1/Rev 1.1/APL1.kicad_sch (KiCad schematic)
At the start: 44 parts, among them J1 6502 BUS, J2 KEYBOARD, J3 SERIAL (DTE), J4 5V DC, J5 PS/2, J6 VIDEO, SW1 POWER, U1 74LS04, U10 ATmega1284-P, U2 6502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

Commit message: Add Rev 1.1
Parts:
- added C17: 10uF, Capacitor_THT:CP_Radial_D4.0mm_P1.50mm, symbol Device:C_Polarized_Small_US
- added R9: 10k, Resistor_THT:R_Axial_DIN0207_L6.3mm_D2.5mm_P10.16mm_Horizontal, symbol Device:R
- R1, R2, R3, R4: value 1k -> 4.7k
Connections:
- net GND: now also C17.2, R9.1
- net VCC: now also C17.1
- net KBDCLRB renamed KBDCLR
- net KBDCLR: now also R9.2
